Commit message: Work on robot model: URDF and meshes. Adding launch file for visualization in RViz

File: src/tractobots_description/urdf/includes/tractobots_materials.urdf.xacro (robot description, xacro)
@@ -8,5 +8,5 @@
   </material>
   <material name="green">
-    <color rgba="0.0 0.8 0.0 1.0"/>
+    <color rgba="${37/255} ${132/255} ${15/255} 1.0"/>
   </material>
   <material name="grey">

File: src/tractobots_description/urdf/includes/tractobots_model.urdf.xacro (robot description, xacro)
@@ -2,31 +2,7 @@
 <robot name="tractobots_model" xmlns:xacro="http://ros.org/wiki/xacro">
   <xacro:include filename="$(find tractobots_description)/urdf/includes/tractobots_properties.urdf.xacro" />
-  <xacro:macro name="wheel" params="name width radius mass">
-    <link name="${name}">
-      <collision>
-        <origin xyz="0 0 0" rpy="${M_PI/2} 0 0"/>
-        <geometry>
-          <cylinder length="${width}" radius="${radius}" />
-        </geometry>
-      </collision>
-      <visual>
-        <origin xyz="0 0 0" rpy="${M_PI/2} 0 0"/>
-        <geometry>
-          <cylinder length="${width}" radius="${radius}" />
-        </geometry>
-        <material name="dark_grey"/>
-      </visual>
-      <inertial>
-        <origin xyz="0 0 0" rpy="${M_PI/2} 0 0"/>
-        <mass value="${mass}"/>
-        <inertia ixx="${1/12*mass*(3*radius*radius + width*width)}" ixy="0.0" ixz="0.0"
-                       iyy="${1/12*mass*(3*radius*radius + width*width)}" iyz="0.0"
-                       izz="${1/2*mass*radius*radius}"/>
-      </inertial>
-    </link>
-  </xacro:macro>
   <!-- Links -->
   <link name="base_link"/>
-  <link name="chassis">
+  <link name="chassis_link">
     <inertial>
       <origin xyz="0 0 0" rpy="0 0 0"/>
@@ -50,33 +26,149 @@
     </collision>
   </link>
-  <xacro:wheel name="front_right_wheel"  width="${front_wheel_width}" radius="${front_wheel_radius}" mass="${front_wheel_mass}"/>
-  <xacro:wheel name="front_left_wheel"   width="${front_wheel_width}" radius="${front_wheel_radius}" mass="${front_wheel_mass}"/>
-  <xacro:wheel name="rear_right_wheel"   width="${rear_wheel_width}"  radius="${rear_wheel_radius}"  mass="${rear_wheel_mass}"/>
-  <xacro:wheel name="rear_left_wheel"    width="${rear_wheel_width}"  radius="${rear_wheel_radius}"  mass="${rear_wheel_mass}"/>
+  <link name="over_chassis_link">
+    <collision>
+      <origin xyz="0 0 0" rpy="0 0 ${M_PI}"/>
+      <geometry>
+        <mesh filename="package://tractobots_description/meshes/over_chassis.stl"/>
+      </geometry>
+    </collision>
+    <visual>
+      <origin xyz="0 0 0" rpy="0 0 ${M_PI}"/>
+      <geometry>
+        <mesh filename="package://tractobots_description/meshes/over_chassis.stl"/>
+      </geometry>
+      <material name="green"/>
+    </visual>
+  </link>
+  <link name="imu_link">
+    <collision>
+      <origin xyz="0 0 0" rpy="0 0 0"/>
+      <geometry>
+        <box size="0.05 0.05 0.05"/>
+      </geometry>
+    </collision>
+    <visual>
+      <origin xyz="0 0 0" rpy="0 0 0"/>
+      <geometry>
+        <box size="0.05 0.05 0.05"/>
+      </geometry>
+      <material name="blue"/>
+    </visual>
+  </link>
+  <link name="gps_link">
+    <collision>
+      <origin xyz="0 0 0" rpy="0 0 0"/>
+      <geometry>
+        <box size="0.05 0.05 0.05"/>
+      </geometry>
+    </collision>
+    <visual>
+      <origin xyz="0 0 0" rpy="0 0 0"/>
+      <geometry>
+        <box size="0.05 0.05 0.05"/>
+      </geometry>
+      <material name="light_grey"/>
+    </visual>
+  </link>
+  <link name="rear_left_wheel_link">
+    <collision>
+      <origin xyz="0 0 0" rpy="${M_PI/2} 0 0"/>
+      <geometry>
+        <mesh filename="package://tractobots_description/meshes/rear_left_wheel.stl"/>
+      </geometry>
+    </collision>
+    <visual>
+      <origin xyz="0 0 0" rpy="${M_PI/2} 0 0"/>
+      <geometry>
+        <mesh filename="package://tractobots_description/meshes/rear_left_wheel.stl"/>
+      </geometry>
+      <material name="dark_grey"/>
+    </visual>
+  </link>
+  <link name="rear_right_wheel_link">
+    <collision>
+      <origin xyz="0 0 0" rpy="${M_PI/2} 0 0"/>
+      <geometry>
+        <mesh filename="package://tractobots_description/meshes/rear_right_wheel.stl"/>
+      </geometry>
+    </collision>
+    <visual>
+      <origin xyz="0 0 0" rpy="${M_PI/2} 0 0"/>
+      <geometry>
+        <mesh filename="package://tractobots_description/meshes/rear_right_wheel.stl"/>
+      </geometry>
+      <material name="dark_grey"/>
+    </visual>
+  </link>
+  <link name="front_left_wheel_link">
+    <collision>
+      <origin xyz="0 0 0" rpy="${M_PI/2} 0 0"/>
+      <geometry>
+        <mesh filename="package://tractobots_description/meshes/front_left_wheel.stl"/>
+      </geometry>
+    </collision>
+    <visual>
+      <origin xyz="0 0 0" rpy="${M_PI/2} 0 0"/>
+      <geometry>
+        <mesh filename="package://tractobots_description/meshes/front_left_wheel.stl"/>
+      </geometry>
+      <material name="dark_grey"/>
+    </visual>
+  </link>
+  <link name="front_right_wheel_link">
+    <collision>
+      <origin xyz="0 0 0" rpy="${M_PI/2} 0 0"/>
+      <geometry>
+        <mesh filename="package://tractobots_description/meshes/front_right_wheel.stl"/>
+      </geometry>
+    </collision>
+    <visual>
+      <origin xyz="0 0 0" rpy="${M_PI/2} 0 0"/>
+      <geometry>
+        <mesh filename="package://tractobots_description/meshes/front_right_wheel.stl"/>
+      </geometry>
+      <material name="dark_grey"/>
+    </visual>
+  </link>
   <!-- Joints -->
   <joint name="chassis_joint" type="fixed">
     <parent link="base_link"/>
-    <child link="chassis"/>
-    <origin xyz="0 0 1.0" rpy="0 0 0"/>
+    <child link="chassis_link"/>
+    <origin xyz="0 0 ${front_wheel_radius}" rpy="0 0 0"/>
+  </joint>
+  <joint name="over_chassis_joint" type="fixed">
+    <parent link="chassis_link"/>
+    <child link="over_chassis_link"/>
+    <origin xyz="0 0 ${chassis_height}" rpy="0 0 0"/>
+  </joint>
+  <joint name="imu_joint" type="fixed">
+    <parent link="over_chassis_link"/>
+    <child link="imu_link"/>
+    <origin xyz="0 0 0"/> <!-- Need to be set! -->
+  </joint>
+  <joint name="gps_joint" type="fixed">
+    <parent link="over_chassis_link"/>
+    <child link="gps_link"/>
+    <origin xyz="0 0 0"/> <!-- Need to be set! -->
   </joint>
   <joint name="front_right_wheel_joint" type="fixed">
-    <parent link="chassis"/>
-    <child link="front_right_wheel"/>
-    <origin xyz="${chassis_length/2} ${front_wheel_width/2 + chassis_width/2} 0" rpy="0 0 0"/>
+    <parent link="chassis_link"/>
+    <child link="front_right_wheel_link"/>
+    <origin xyz="${chassis_length/2} ${chassis_width/2} 0" rpy="0 0 0"/>
   </joint>
   <joint name="front_left_wheel_joint" type="fixed">
-    <parent link="chassis"/>
-    <child link="front_left_wheel"/>
-    <origin xyz="${chassis_length/2} ${-(front_wheel_width/2 + chassis_width/2)} 0" rpy="0 0 0"/>
+    <parent link="chassis_link"/>
+    <child link="front_left_wheel_link"/>
+    <origin xyz="${chassis_length/2} ${-(chassis_width/2)} 0" rpy="0 0 0"/>
   </joint>
   <joint name="rear_right_wheel_joint" type="fixed">
-    <parent link="chassis"/>
-    <child link="rear_right_wheel"/>
-    <origin xyz="${-chassis_length/2} ${rear_wheel_width/2 + chassis_width/2} ${-(front_wheel_radius - rear_wheel_radius)}" rpy="0 0 0"/>
+    <parent link="chassis_link"/>
+    <child link="rear_right_wheel_link"/>
+    <origin xyz="${-chassis_length/2} ${chassis_width/2} ${-(front_wheel_radius - rear_wheel_radius)}" rpy="0 0 0"/>
   </joint>
   <joint name="rear_left_wheel_joint" type="fixed">
-    <parent link="chassis"/>
-    <child link="rear_left_wheel"/>
-    <origin xyz="${-chassis_length/2} ${-(rear_wheel_width/2 + chassis_width/2)} ${-(front_wheel_radius - rear_wheel_radius)}" rpy="0 0 0"/>
+    <parent link="chassis_link"/>
+    <child link="rear_left_wheel_link"/>
+    <origin xyz="${-chassis_length/2} ${-(chassis_width/2)} ${-(front_wheel_radius - rear_wheel_radius)}" rpy="0 0 0"/>
   </joint>
 </robot>

File: src/tractobots_description/urdf/includes/tractobots_properties.urdf.xacro (robot description, xacro)
@@ -3,17 +3,18 @@
   <xacro:property name="M_PI" 				 value="3.1415926535897931"/>
   <!-- Constants for chassis -->
-  <xacro:property name="chassis_height" 		 value="0.3"/>
-  <xacro:property name="chassis_length" 		 value="0.5"/>
-  <xacro:property name="chassis_width"  		 value="0.4"/>
+  <xacro:property name="chassis_height" 		 value="0.001"/>
+  <xacro:property name="chassis_length" 		 value="2.4"/>
+  <xacro:property name="chassis_width"  		 value="1.348"/>
   <xacro:property name="chassis_mass"   		 value="20" />
-  <!-- Constants for front wheels -->
-  <xacro:property name="front_wheel_radius" 		 value="0.2"/>
-  <xacro:property name="front_wheel_width"  		 value="0.1"/>
-  <xacro:property name="front_wheel_mass"   		 value="4"/>
-  <xacro:property name="front_wheel_track"  		 value="0.6"/>
-  <!-- Constants for rear wheels -->
-  <xacro:property name="rear_wheel_radius" 		 value="0.12"/>
-  <xacro:property name="rear_wheel_width" 		 value="0.08"/>
-  <xacro:property name="rear_wheel_mass"  		 value="2"/>
-  <xacro:property name="rear_wheel_track" 		 value="0.535"/>
+  <!-- Data for wheel dimensions from: http://agri.firestone.eu/down/FS_AGDatabook2016_Brochure_EU.pdf -->
+  <!-- Constants for front wheels (320/85R24) -->
+  <xacro:property name="front_wheel_radius" 		 value="0.575"/>
+  <xacro:property name="front_wheel_width"  		 value="0.313"/>
+  <xacro:property name="front_wheel_mass"   		 value="4"/> <!-- Must be calculated -->
+  <xacro:property name="front_wheel_track"  		 value="0.6"/> <!-- Must be calculated -->
+  <!-- Constants for rear wheels (460/85R30) -->
+  <xacro:property name="rear_wheel_radius"     value="0.768"/>
+  <xacro:property name="rear_wheel_width"      value="0.484"/>
+  <xacro:property name="rear_wheel_mass"       value="2"/> <!-- Must be calculated -->
+  <xacro:property name="rear_wheel_track"      value="0.535"/> <!-- Must be calculated -->
 </robot>
